File: Schematic files/LCDLayer/LCD Layer_sch.kicad_sch (KiCad schematic)
At the start: 2 parts

Commit message: Finished Schematic
Connections:
- net +3V3: no longer J4.10 (LEDA)
- now unconnected: J4.11 (LEDK1), J4.12 (LEDK2), J4.13 (LEDK3), J4.14 (LEDK4)
- no-connect marks 5 -> 9
Other:
- company: (none) -> Sidharth Sreeram
- title: (none) -> LCD_Panel
Changed lines of the file:
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@@
 (kicad_sch (version 20230121) (generator eeschema)
   (paper "A4")
-  (junction (at 87.63 68.58) (diameter 0) (color 0 0 0 0)
-  )
-  (junction (at 87.63 73.66) (diameter 0) (color 0 0 0 0)
+  (title_block
+    (title "LCD_Panel")
+    (date "2024-02-27")
+    (rev "1.0")
+    (company "Sidharth Sreeram")
   )
   (junction (at 120.65 53.34) (diameter 0) (color 0 0 0 0)
   )
-  (junction (at 96.52 63.5) (diameter 0) (color 0 0 0 0)
-  )
-  (junction (at 87.63 71.12) (diameter 0) (color 0 0 0 0)
-  )
+  (no_connect (at 87.63 66.04))
+  (no_connect (at 87.63 71.12))
   (no_connect (at 87.63 86.36))
+  (no_connect (at 87.63 73.66))
   (no_connect (at 87.63 83.82))
+  (no_connect (at 87.63 76.2))
   (no_connect (at 87.63 78.74))
+  (no_connect (at 87.63 68.58))
   (no_connect (at 87.63 81.28))
-  (no_connect (at 97.79 69.85))
   (wire (pts (xy 101.6 55.88) (xy 107.95 55.88))
     (stroke (width 0) (type default))
@@
     (stroke (width 0) (type default))
   )
-  (wire (pts (xy 87.63 68.58) (xy 97.79 68.58))
-    (stroke (width 0) (type default))
-  )
-  (wire (pts (xy 96.52 63.5) (xy 115.57 63.5))
+  (wire (pts (xy 87.63 63.5) (xy 115.57 63.5))
     (stroke (width 0) (type default))
   )
   (wire (pts (xy 87.63 43.18) (xy 87.63 38.1))
-    (stroke (width 0) (type default))
-  )
-  (wire (pts (xy 87.63 63.5) (xy 96.52 63.5))
     (stroke (width 0) (type default))
   )
@@
     (stroke (width 0) (type default))
   )
-  (wire (pts (xy 87.63 68.58) (xy 87.63 71.12))
-    (stroke (width 0) (type default))
-  )
-  (wire (pts (xy 96.52 63.5) (xy 96.52 66.04))
-    (stroke (width 0) (type default))
-  )
   (wire (pts (xy 107.95 55.88) (xy 107.95 57.15))
-    (stroke (width 0) (type default))
-  )
-  (wire (pts (xy 96.52 66.04) (xy 87.63 66.04))
     (stroke (width 0) (type default))
   )
@@
     (stroke (width 0) (type default))
   )
-  (wire (pts (xy 97.79 68.58) (xy 97.79 69.85))
-    (stroke (width 0) (type default))
-  )
-  (wire (pts (xy 87.63 73.66) (xy 87.63 76.2))
-    (stroke (width 0) (type default))
-  )
-  (wire (pts (xy 87.63 73.66) (xy 87.63 71.12))
-    (stroke (width 0) (type default))
+  (rectangle (start 40.64 30.48) (end 151.13 100.33)
+    (stroke (width 0) (type dash))
+    (fill (type none))
   )
   (text "Backlight LED's\n" (at 91.44 73.66 0)
