File: Schematic files/LCDLayer/LCDLayer.kicad_sch (KiCad schematic)
At the start: 0 parts

Commit message: Finished Schematic
Other:
- sheet LCD Layer renamed LCD_Panel
- sheet MotorController renamed Motor_Controller
- sheet Power renamed Power_Management
- sheet Processor renamed STM32F103C8T6_MCU
- sheet USBReader renamed USBReader & SDCard
- sheet UVLight renamed UVLED_Panel
- note added: "GND +12V +5V +3V3 SPI GPIO"
- company: (none) -> Sidharth Sreeram
- title: (none) -> Resin 3D Printer PCB
Changed lines of the file:
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@@
 (kicad_sch (version 20230121) (generator eeschema)
   (paper "A4")
-  (sheet (at 233.68 55.88) (size 15.24 11.43) (fields_autoplaced)
-    (stroke (width 0.1524) (type solid))
-    (fill (color 0 0 0 0.0000))
-    (property "Sheetname" "buck converter" (at 233.68 55.1684 0)
+  (title_block
+    (title "Resin 3D Printer PCB")
+    (date "2024-02-27")
+    (rev "1.0")
+    (company "Sidharth Sreeram")
+  )
+  (bus (pts (xy 29.21 34.29) (xy 40.64 34.29))
+    (stroke (width 2) (type default) (color 194 0 194 1))
+  )
+  (bus (pts (xy 29.21 116.84) (xy 29.21 34.29))
+    (stroke (width 2) (type default) (color 194 0 194 1))
+  )
+  (bus (pts (xy 146.05 68.58) (xy 170.18 68.58))
+    (stroke (width 1) (type default) (color 0 255 0 1))
+  )
+  (bus (pts (xy 207.01 96.52) (xy 207.01 116.84))
+    (stroke (width 2) (type default) (color 0 0 0 1))
+  )
+  (bus (pts (xy 35.56 40.64) (xy 40.64 40.64))
+    (stroke (width 2) (type default) (color 0 0 0 1))
+  )
+  (bus (pts (xy 232.41 25.4) (xy 210.82 25.4))
+    (stroke (width 2) (type default) (color 0 0 0 1))
+  )
+  (wire (pts (xy 26.67 173.99) (xy 39.37 173.99))
+    (stroke (width 2) (type default) (color 194 0 194 1))
+  )
+  (wire (pts (xy 26.67 180.34) (xy 39.37 180.34))
+    (stroke (width 2) (type default) (color 255 153 0 1))
+  )
+  (bus (pts (xy 223.52 35.56) (xy 223.52 116.84))
+    (stroke (width 2) (type default) (color 255 153 0 1))
+  )
+  (bus (pts (xy 35.56 116.84) (xy 35.56 40.64))
+    (stroke (width 2) (type default) (color 0 0 0 1))
+  )
+  (wire (pts (xy 26.67 186.69) (xy 39.37 186.69))
+    (stroke (width 2) (type default) (color 128 77 0 1))
+  )
+  (bus (pts (xy 223.52 35.56) (xy 210.82 35.56))
+    (stroke (width 2) (type default) (color 255 153 0 1))
+  )
+  (bus (pts (xy 80.01 71.12) (xy 97.79 71.12))
+    (stroke (width 1) (type default) (color 0 255 0 1))
+  )
+  (bus (pts (xy 80.01 68.58) (xy 97.79 68.58))
+    (stroke (width 1) (type default) (color 0 255 0 1))
+  )
+  (wire (pts (xy 26.67 167.64) (xy 39.37 167.64))
+    (stroke (width 2) (type default) (color 255 0 0 1))
+  )
+  (bus (pts (xy 80.01 25.4) (xy 97.79 25.4))
+    (stroke (width 1) (type default) (color 0 255 0 1))
+  )
+  (bus (pts (xy 80.01 44.45) (xy 97.79 44.45))
+    (stroke (width 2) (type default) (color 128 77 0 1))
+  )
+  (wire (pts (xy 40.64 27.94) (xy 22.86 27.94))
+    (stroke (width 2) (type default) (color 255 153 0 1))
+  )
+  (bus (pts (xy 80.01 27.94) (xy 97.79 27.94))
+    (stroke (width 1) (type default) (color 0 255 0 1))
+  )
+  (wire (pts (xy 26.67 161.29) (xy 39.37 161.29))
+    (stroke (width 2) (type default) (color 0 0 0 1))
+  )
+  (wire (pts (xy 22.86 27.94) (xy 22.86 116.84))
+    (stroke (width 2) (type default) (color 255 153 0 1))
+  )
+  (wire (pts (xy 26.67 193.04) (xy 39.37 193.04))
+    (stroke (width 1) (type default) (color 0 255 0 1))
+  )
+  (bus (pts (xy 232.41 25.4) (xy 232.41 116.84))
+    (stroke (width 2) (type default) (color 0 0 0 1))
+  )
+  (bus (pts (xy 44.45 90.17) (xy 44.45 116.84))
+    (stroke (width 2) (type default) (color 0 0 0 1))
+  )
+  (bus (pts (xy 80.01 73.66) (xy 97.79 73.66))
+    (stroke (width 1) (type default) (color 0 255 0 1))
+  )
+  (bus (pts (xy 49.53 90.17) (xy 49.53 116.84))
+    (stroke (width 2) (type default) (color 255 0 0 1))
+  )
+  (bus (pts (xy 146.05 29.21) (xy 170.18 29.21))
+    (stroke (width 2) (type default) (color 128 77 0 1))
+  )
+  (bus (pts (xy 80.01 76.2) (xy 97.79 76.2))
+    (stroke (width 1) (type default) (color 0 255 0 1))
+  )
+  (bus (pts (xy 109.22 95.25) (xy 109.22 116.84))
+    (stroke (width 2) (type default) (color 255 0 0 1))
+  )
+  (bus (pts (xy 198.12 96.52) (xy 198.12 116.84))
+    (stroke (width 2) (type default) (color 255 0 0 1))
+  )
+  (bus (pts (xy 135.89 95.25) (xy 135.89 116.84))
+    (stroke (width 2) (type default) (color 255 153 0 1))
+  )
+  (bus (pts (xy 80.01 78.74) (xy 97.79 78.74))
+    (stroke (width 1) (type default) (color 0 255 0 1))
+  )
+  (rectangle (start 21.59 156.21) (end 115.57 195.58)
+    (stroke (width 0) (type default))
+    (fill (type none))
+  )
+  (text "GND\n\n+12V\n\n+5V\n\n+3V3\n\nSPI\n\nGPIO" (at 41.91 194.31 0)
+    (effects (font (size 2 2)) (justify left bottom))
+  )
+  (sheet (at 264.16 16.51) (size 15.24 11.43) (fields_autoplaced)
+    (stroke (width 0.1524) (type solid))
+    (fill (color 0 0 0 0.0000))
+    (property "Sheetname" "buck converter" (at 264.16 15.7984 0)
       (effects (font (size 1.27 1.27)) (justify left bottom))
     )
-    (property "Sheetfile" "buckconvert.kicad_sch" (at 233.68 67.8946 0)
+    (property "Sheetfile" "buckconvert.kicad_sch" (at 264.16 28.5246 0)
       (effects (font (size 1.27 1.27)) (justify left top))
     )
@@
     )
   )
-  (sheet (at 204.47 97.79) (size 41.91 35.56) (fields_autoplaced)
-    (stroke (width 0.1524) (type solid))
-    (fill (color 0 0 0 0.0000))
-    (property "Sheetname" "Power" (at 204.47 97.0784 0)
-      (effects (font (size 1.27 1.27)) (justify left bottom))
-    )
-    (property "Sheetfile" "Power.kicad_sch" (at 204.47 133.9346 0)
+  (sheet (at 21.59 116.84) (size 238.76 35.56)
+    (stroke (width 0.1524) (type solid))
+    (fill (color 0 0 0 0.0000))
+    (property "Sheetname" "Power_Management" (at 22.86 125.73 0)
+      (effects (font (size 5 5) bold) (justify left bottom))
+    )
+    (property "Sheetfile" "Power.kicad_sch" (at 22.86 149.86 0)
       (effects (font (size 1.27 1.27)) (justify left top))
     )
@@
     )
   )
-  (sheet (at 167.64 21.59) (size 40.64 34.29) (fields_autoplaced)
-    (stroke (width 0.1524) (type solid))
-    (fill (color 0 0 0 0.0000))
-    (property "Sheetname" "LCD Layer" (at 167.64 20.8784 0)
-      (effects (font (size 1.27 1.27)) (justify left bottom))
-    )
-    (property "Sheetfile" "LCD Layer_sch.kicad_sch" (at 167.64 56.4646 0)
+  (sheet (at 170.18 19.05) (size 40.64 33.02)
+    (stroke (width 0.1524) (type solid))
+    (fill (color 0 0 0 0.0000))
+    (property "Sheetname" "LCD_Panel" (at 171.45 22.86 0)
+      (effects (font (size 2 2) bold) (justify left bottom))
+    )
+    (property "Sheetfile" "LCD Layer_sch.kicad_sch" (at 171.45 50.8 0)
       (effects (font (size 1.27 1.27)) (justify left top))
     )
@@
     )
   )
-  (sheet (at 100.33 31.75) (size 34.29 36.83) (fields_autoplaced)
-    (stroke (width 0.1524) (type solid))
-    (fill (color 0 0 0 0.0000))
-    (property "Sheetname" "Processor" (at 100.33 31.0384 0)
-      (effects (font (size 1.27 1.27)) (justify left bottom))
-    )
-    (property "Sheetfile" "Processor.kicad_sch" (at 100.33 69.1646 0)
+  (sheet (at 97.79 19.05) (size 48.26 76.2)
+    (stroke (width 0.1524) (type solid))
+    (fill (color 0 0 0 0.0000))
+    (property "Sheetname" "STM32F103C8T6_MCU" (at 99.06 22.86 0)
+      (effects (font (size 2 2) bold) (justify left bottom))
+    )
+    (property "Sheetfile" "Processor.kicad_sch" (at 99.06 91.44 0)
       (effects (font (size 1.27 1.27)) (justify left top))
     )
@@
     )
   )
-  (sheet (at 109.22 107.95) (size 39.37 26.67) (fields_autoplaced)
-    (stroke (width 0.1524) (type solid))
-    (fill (color 0 0 0 0.0000))
-    (property "Sheetname" "MotorController" (at 109.22 107.2384 0)
-      (effects (font (size 1.27 1.27)) (justify left bottom))
-    )
-    (property "Sheetfile" "MotorController.kicad_sch" (at 109.22 135.2046 0)
+  (sheet (at 40.64 63.5) (size 39.37 26.67)
+    (stroke (width 0.1524) (type solid))
+    (fill (color 0 0 0 0.0000))
+    (property "Sheetname" "Motor_Controller" (at 40.64 67.31 0)
+      (effects (font (size 2 2) bold) (justify left bottom))
+    )
+    (property "Sheetfile" "MotorController.kicad_sch" (at 41.91 87.63 0)
       (effects (font (size 1.27 1.27)) (justify left top))
     )
@@
     )
   )
-  (sheet (at 41.91 102.87) (size 39.37 30.48) (fields_autoplaced)
-    (stroke (width 0.1524) (type solid))
-    (fill (color 0 0 0 0.0000))
-    (property "Sheetname" "USBReader" (at 41.91 102.1584 0)
-      (effects (font (size 1.27 1.27)) (justify left bottom))
-    )
-    (property "Sheetfile" "USBReader.kicad_sch" (at 41.91 133.9346 0)
+  (sheet (at 40.64 17.78) (size 39.37 30.48)
+    (stroke (width 0.1524) (type solid))
+    (fill (color 0 0 0 0.0000))
+    (property "Sheetname" "USBReader & SDCard" (at 40.64 21.59 0)
+      (effects (font (size 2 2) bold) (justify left bottom))
+    )
+    (property "Sheetfile" "USBReader.kicad_sch" (at 41.91 45.72 0)
       (effects (font (size 1.27 1.27)) (justify left top))
     )
@@
     )
   )
-  (sheet (at 26.67 22.86) (size 45.72 41.91) (fields_autoplaced)
-    (stroke (width 0.1524) (type solid))
-    (fill (color 0 0 0 0.0000))
-    (property "Sheetname" "UVLight" (at 26.67 22.1484 0)
-      (effects (font (size 1.27 1.27)) (justify left bottom))
-    )
-    (property "Sheetfile" "UVLight.kicad_sch" (at 26.67 65.3546 0)
-      (effects (font (size 1.27 1.27)) (justify left top))
-    )
+  (sheet (at 170.18 59.69) (size 40.64 36.83)
+    (stroke (width 0.1524) (type solid))
+    (fill (color 0 0 0 0.0000))
+    (property "Sheetname" "UVLED_Panel" (at 171.45 63.5 0)
+      (effects (font (size 2 2) bold) (justify left bottom))
+    )
+    (property "Sheetfile" "UVLight.kicad_sch" (at 171.45 93.98 0)
+      (effects (font (size 1.27 1.27)) (justify left top))
+    )
