File: Schematic files/LCDLayer/MotorController.kicad_sch (KiCad schematic)
At the start: 5 parts, among them M1 Z-Axis Stepper Motor

Commit message: Finished Schematic
Other:
- company: (none) -> Sidharth Sreeram
- title: (none) -> Motor_Controller
Changed lines of the file:
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@@
 (kicad_sch (version 20230121) (generator eeschema)
   (paper "A4")
+  (title_block
+    (title "Motor_Controller")
+    (date "2024-02-27")
+    (rev "1.0")
+    (company "Sidharth Sreeram")
+  )
   (junction (at 134.62 86.36) (diameter 0) (color 0 0 0 0)
   )
