File: Schematic files/LCDLayer/Power.kicad_sch (KiCad schematic)
At the start: 10 parts, among them J5 Mini-DIN-5, U3 LD1117S33TR_SOT223

Commit message: Finished Schematic
Parts:
- added F1: 500mA, symbol Device:Fuse
Connections:
- net +12V: now also D39.2 (A); no longer R20.1
- net +3V3: now also F1.2; no longer D40.1 (K)
- net +5V: now also D38.2 (A); no longer R19.1
- net GND: now also R19.2, R20.1, R21.1; no longer D38.1 (K), D39.1 (K)
- net at C6.1, U3.2 (VO): now also D40.2 (A), F1.1; no longer R21.1
- net at R20.2: now also D39.1 (K); no longer D39.2 (A)
- net at R21.2: now also D40.1 (K); no longer D40.2 (A)
- new net: D38.1 (K), R19.1
Other:
- company: (none) -> Sidharth Sreeram
- title: (none) -> Power_Management
- moved on the sheet: C5, C6, D38, D39, D40, R19, R20, R21, U3
