File: Schematic files/LCDLayer/USBReader.kicad_sch (KiCad schematic)
At the start: 5 parts, among them J2 SD_Card, J3 USB_A

Commit message: Finished Schematic
Parts:
- added C8: 100nC, symbol Device:C
Connections:
- net +3V3: now also C8.1
- net GND: now also C8.2
Other:
- company: (none) -> Sidharth Sreeram
- title: (none) -> USBReader & SDCard
- moved on the sheet: R8
Changed lines of the file:
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@@
 (kicad_sch (version 20230121) (generator eeschema)
   (paper "A4")
+  (title_block
+    (title "USBReader & SDCard")
+    (date "2024-02-27")
+    (rev "1.0")
+    (company "Sidharth Sreeram")
+  )
+  (junction (at 137.16 62.23) (diameter 0) (color 0 0 0 0)
+  )
   (junction (at 177.8 48.26) (diameter 0) (color 0 0 0 0)
   )
   (junction (at 58.42 57.15) (diameter 0) (color 0 0 0 0)
   )
+  (junction (at 125.73 54.61) (diameter 0) (color 0 0 0 0)
+  )
+  (junction (at 125.73 62.23) (diameter 0) (color 0 0 0 0)
+  )
   (no_connect (at 182.88 45.72))
   (no_connect (at 182.88 66.04))
@@
     (stroke (width 0) (type default))
   )
-  (wire (pts (xy 153.67 55.88) (xy 182.88 55.88))
-    (stroke (width 0) (type default))
-  )
-  (wire (pts (xy 139.7 58.42) (xy 140.97 58.42))
+  (wire (pts (xy 153.67 58.42) (xy 154.94 58.42))
     (stroke (width 0) (type default))
   )
@@
     (stroke (width 0) (type default))
   )
-  (wire (pts (xy 153.67 50.8) (xy 153.67 55.88))
+  (wire (pts (xy 125.73 50.8) (xy 125.73 54.61))
     (stroke (width 0) (type default))
   )
@@
     (stroke (width 0) (type default))
   )
-  (wire (pts (xy 182.88 60.96) (xy 154.94 60.96))
+  (wire (pts (xy 177.8 48.26) (xy 182.88 48.26))
     (stroke (width 0) (type default))
   )
-  (wire (pts (xy 177.8 48.26) (xy 182.88 48.26))
+  (wire (pts (xy 139.7 52.07) (xy 139.7 54.61))
     (stroke (width 0) (type default))
   )
-  (wire (pts (xy 182.88 53.34) (xy 151.13 53.34))
+  (wire (pts (xy 162.56 62.23) (xy 162.56 60.96))
     (stroke (width 0) (type default))
   )
@@
     (stroke (width 0) (type default))
   )
+  (wire (pts (xy 161.29 53.34) (xy 161.29 49.53))
+    (stroke (width 0) (type default))
+  )
   (wire (pts (xy 58.42 57.15) (xy 74.93 57.15))
     (stroke (width 0) (type default))
   )
-  (wire (pts (xy 148.59 58.42) (xy 182.88 58.42))
+  (wire (pts (xy 162.56 58.42) (xy 182.88 58.42))
+    (stroke (width 0) (type default))
+  )
+  (wire (pts (xy 125.73 62.23) (xy 137.16 62.23))
     (stroke (width 0) (type default))
   )
@@
     (stroke (width 0) (type default))
   )
+  (wire (pts (xy 125.73 54.61) (xy 139.7 54.61))
+    (stroke (width 0) (type default))
+  )
+  (wire (pts (xy 162.56 60.96) (xy 182.88 60.96))
+    (stroke (width 0) (type default))
+  )
+  (wire (pts (xy 137.16 49.53) (xy 137.16 62.23))
+    (stroke (width 0) (type default))
+  )
   (wire (pts (xy 176.53 50.8) (xy 182.88 50.8))
     (stroke (width 0) (type default))
   )
-  (wire (pts (xy 154.94 60.96) (xy 154.94 71.12))
+  (wire (pts (xy 182.88 55.88) (xy 160.02 55.88))
+    (stroke (width 0) (type default))
+  )
+  (wire (pts (xy 182.88 53.34) (xy 161.29 53.34))
+    (stroke (width 0) (type default))
+  )
+  (wire (pts (xy 160.02 55.88) (xy 160.02 52.07))
+    (stroke (width 0) (type default))
+  )
+  (wire (pts (xy 125.73 62.23) (xy 125.73 67.31))
+    (stroke (width 0) (type default))
+  )
+  (wire (pts (xy 137.16 62.23) (xy 162.56 62.23))
+    (stroke (width 0) (type default))
+  )
+  (wire (pts (xy 161.29 49.53) (xy 137.16 49.53))
+    (stroke (width 0) (type default))
+  )
+  (wire (pts (xy 160.02 52.07) (xy 139.7 52.07))
     (stroke (width 0) (type default))
   )
@@
     )
   )
-  (text "SD_Card_Connections" (at 120.65 31.75 0)
+  (text "SD_Card_Connections" (at 120.65 33.02 0)
     (effects (font (size 1.27 1.27)) (justify left bottom))
   )
@@
     (effects (font (size 1.27 1.27)) (justify left bottom))
   )
-  (global_label "SD_CS" (shape bidirectional) (at 173.99 48.26 180) (fields_autoplaced)
+  (global_label "SD_CS" (shape input) (at 173.99 48.26 180) (fields_autoplaced)
     (effects (font (size 1.27 1.27)) (justify right))
-    (property "Intersheetrefs" "${INTERSHEET_REFS}" (at 163.9669 48.26 0)
+    (property "Intersheetrefs" "${INTERSHEET_REFS}" (at 165.0782 48.26 0)
       (effects (font (size 1.27 1.27)) (justify right) hide)
     )
   )
-  (global_label "SPI_2_MOSI" (shape bidirectional) (at 176.53 50.8 180) (fields_autoplaced)
+  (global_label "SPI_2_MOSI" (shape input) (at 176.53 50.8 180) (fields_autoplaced)
     (effects (font (size 1.27 1.27)) (justify right))
-    (property "Intersheetrefs" "${INTERSHEET_REFS}" (at 161.6083 50.8 0)
+    (property "Intersheetrefs" "${INTERSHEET_REFS}" (at 162.7196 50.8 0)
       (effects (font (size 1.27 1.27)) (justify right) hide)
     )
   )
-  (global_label "SPI_2_SCLK" (shape input) (at 139.7 58.42 180) (fields_autoplaced)
+  (global_label "SPI_2_SCLK" (shape input) (at 153.67 58.42 180) (fields_autoplaced)
     (effects (font (size 1.27 1.27)) (justify right))
-    (property "Intersheetrefs" "${INTERSHEET_REFS}" (at 125.7082 58.42 0)
+    (property "Intersheetrefs" "${INTERSHEET_REFS}" (at 139.6782 58.42 0)
       (effects (font (size 1.27 1.27)) (justify right) hide)
     )
   )
-  (global_label "SPI_2_MISO" (shape bidirectional) (at 180.34 63.5 180) (fields_autoplaced)
+  (global_label "SPI_2_MISO" (shape output) (at 180.34 63.5 180) (fields_autoplaced)
     (effects (font (size 1.27 1.27)) (justify right))
-    (property "Intersheetrefs" "${INTERSHEET_REFS}" (at 165.4183 63.5 0)
+    (property "Intersheetrefs" "${INTERSHEET_REFS}" (at 166.5296 63.5 0)
       (effects (font (size 1.27 1.27)) (justify right) hide)
     )
@@
     )
   )
-  (symbol (lib_id "Device:R_US") (at 144.78 58.42 90) (unit 1)
-    (in_bom yes) (on_board yes) (dnp no) (fields_autoplaced)
-    (property "Reference" "R8" (at 144.78 52.07 90)
+  (symbol (lib_id "Device:R_US") (at 158.75 58.42 90) (unit 1)
+    (in_bom yes) (on_board yes) (dnp no)
+    (property "Reference" "R8" (at 157.48 54.61 90)
       (effects (font (size 1.27 1.27)))
     )
-    (property "Value" "1kR" (at 144.78 54.61 90)
+    (property "Value" "1kR" (at 157.7709 56.3974 90)
       (effects (font (size 1.27 1.27)))
     )
-    (property "Footprint" "" (at 145.034 57.404 90)
+    (property "Footprint" "" (at 159.004 57.404 90)
       (effects (font (size 1.27 1.27)) hide)
     )
-    (property "Datasheet" "~" (at 144.78 58.42 0)
+    (property "Datasheet" "~" (at 158.75 58.42 0)
       (effects (font (size 1.27 1.27)) hide)
     )
@@
     )
   )
-  (symbol (lib_id "power:GND") (at 151.13 53.34 0) (unit 1)
-    (in_bom yes) (on_board yes) (dnp no)
-    (property "Reference" "#PWR08" (at 151.13 59.69 0)
-      (effects (font (size 1.27 1.27)) hide)
-    )
-    (property "Value" "GND" (at 147.32 60.96 0)
-      (effects (font (size 1.27 1.27)) hide)
-    )
-    (property "Footprint" "" (at 151.13 53.34 0)
-      (effects (font (size 1.27 1.27)) hide)
-    )
-    (property "Datasheet" "" (at 151.13 53.34 0)
-      (effects (font (size 1.27 1.27)) hide)
-    )
-    (pin "1")
-    (instances
-      (project "LCDLayer"
-        (path "/af5d6fb3-2577-4120-8af3-1828a4be58c2/75b4f9cb-929f-4c12-9fb2-570bcc17a11a"
-          (reference "#PWR08") (unit 1)
-        )
-      )
-    )
-  )
   (symbol (lib_id "power:+3V3") (at 58.42 49.53 0) (unit 1)
     (in_bom yes) (on_board yes) (dnp no) (fields_autoplaced)
@@
     )
   )
-  (symbol (lib_id "power:GND") (at 154.94 71.12 0) (unit 1)
+  (symbol (lib_id "Device:C") (at 125.73 58.42 0) (unit 1)
+    (in_bom yes) (on_board yes) (dnp no)
+    (property "Reference" "C8" (at 128.27 57.15 0)
+      (effects (font (size 1.27 1.27)) (justify left))
+    )
+    (property "Value" "100nC" (at 128.27 59.69 0)
+      (effects (font (size 1.27 1.27)) (justify left))
+    )
+    (property "Footprint" "" (at 126.6952 62.23 0)
+      (effects (font (size 1.27 1.27)) hide)
+    )
+    (property "Datasheet" "~" (at 125.73 58.42 0)
+      (effects (font (size 1.27 1.27)) hide)
+    )
+    (pin "1")
+    (pin "2")
+    (instances
+      (project "LCDLayer"
+        (path "/af5d6fb3-2577-4120-8af3-1828a4be58c2/75b4f9cb-929f-4c12-9fb2-570bcc17a11a"
+          (reference "C8") (unit 1)
+        )
+      )
+    )
+  )
+  (symbol (lib_id "power:GND") (at 125.73 67.31 0) (unit 1)
     (in_bom yes) (on_board yes) (dnp no) (fields_autoplaced)
-    (property "Reference" "#PWR010" (at 154.94 77.47 0)
+    (property "Reference" "#PWR010" (at 125.73 73.66 0)
       (effects (font (size 1.27 1.27)) hide)
     )
-    (property "Value" "GND" (at 154.94 76.2 0)
+    (property "Value" "GND" (at 125.73 72.39 0)
       (effects (font (size 1.27 1.27)) hide)
     )
-    (property "Footprint" "" (at 154.94 71.12 0)
+    (property "Footprint" "" (at 125.73 67.31 0)
       (effects (font (size 1.27 1.27)) hide)
     )
-    (property "Datasheet" "" (at 154.94 71.12 0)
+    (property "Datasheet" "" (at 125.73 67.31 0)
       (effects (font (size 1.27 1.27)) hide)
     )
@@
     )
   )
-  (symbol (lib_id "power:+3V3") (at 153.67 50.8 0) (unit 1)
+  (symbol (lib_id "power:+3V3") (at 125.73 50.8 0) (unit 1)
     (in_bom yes) (on_board yes) (dnp no) (fields_autoplaced)
-    (property "Reference" "#PWR09" (at 153.67 54.61 0)
+    (property "Reference" "#PWR09" (at 125.73 54.61 0)
       (effects (font (size 1.27 1.27)) hide)
     )
-    (property "Value" "+3V3" (at 153.67 45.72 0)
+    (property "Value" "+3V3" (at 125.73 45.72 0)
       (effects (font (size 1.27 1.27)))
     )
-    (property "Footprint" "" (at 153.67 50.8 0)
+    (property "Footprint" "" (at 125.73 50.8 0)
       (effects (font (size 1.27 1.27)) hide)
     )
-    (property "Datasheet" "" (at 153.67 50.8 0)
+    (property "Datasheet" "" (at 125.73 50.8 0)
       (effects (font (size 1.27 1.27)) hide)
     )
