File: Schematic files/LCDLayer/buckconvert.kicad_sch (KiCad schematic)
At the start: 11 parts, among them Q2 Q_NMOS_SGD

Commit message: Finished Schematic
Other:
- company: (none) -> Sidharth Sreeram
Changed lines of the file:
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@@
 (kicad_sch (version 20230121) (generator eeschema)
   (paper "A4")
+  (title_block
+    (date "2024-02-27")
+    (rev "1.0")
+    (company "Sidharth Sreeram")
+  )
   (junction (at 121.285 83.82) (diameter 0) (color 0 0 0 0)
   )
