File: Schematic files/Schematics/USBReader.kicad_sch (KiCad schematic)
At the start: 6 parts, among them J3 SD_Card, J4 USB_A

Commit message: pcb
Parts:
- J4: footprint Connector_USB:USB_A_Wuerth_614004134726_Horizontal -> Connector_USB:USB_A_TE_292303-7_Horizontal
Changed lines of the file:
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@@
       (effects (font (size 1.27 1.27)))
     )
-    (property "Footprint" "Connector_USB:USB_A_Wuerth_614004134726_Horizontal" (at 38.1 58.42 0)
+    (property "Footprint" "Connector_USB:USB_A_TE_292303-7_Horizontal" (at 38.1 58.42 0)
       (effects (font (size 1.27 1.27)) hide)
     )
